File: Hardware/Sunflower_Rev1-3.brd (EAGLE design)
At the start: 76.9 x 81.1 mm, 115 parts, among them CN1 2060-452/998-404, CN10 (DNP), CN2 (DNP), CN3 T400 THERMO CLIP, CN4 2908-05WB-M6, CN5 2060-452/998-404TEMP, CN6 1X8M-H7.5, CN7 1X10M-H7.5, CN8 1X8M-H7.5, CN9 2X3F-H7.5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

Commit message: Fix Typo + Add Schematic as PDF
Schematic Typo Corrected.
Electrical Characteristic Updated.
Sunflower Shield PDF Schematic Added.
Parts:
- C31: value 2200pF -> 0.22uF
Changed lines of the file:
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@@
 <attribute name="VALUE" x="62.484" y="61.595" size="0.8128" layer="27" ratio="18" rot="R180"/>
 </element>
-<element name="C31" library="microbuilder" package="0603" value="2200pF" x="56.515" y="53.1495" smashed="yes" rot="R270">
+<element name="C31" library="microbuilder" package="0603" value="0.22uF" x="56.515" y="53.1495" smashed="yes" rot="R270">
 <attribute name="NAME" x="60.198" y="51.562" size="0.8128" layer="25" font="vector" ratio="18" rot="R90"/>
 <attribute name="VALUE" x="55.753" y="51.3715" size="0.8128" layer="27" font="vector" ratio="18" rot="R270"/>
