File: Hardware/Sunflower_Rev1-3.sch (EAGLE design)
At the start: 115 parts, among them CN1 2060-452/998-404, CN10 (DNP), CN2 (DNP), CN3 T400 THERMO CLIP, CN4 2908-05WB-M6, CN5 2060-452/998-404TEMP, CN6 1X8M-H7.5, CN7 1X10M-H7.5, CN8 1X8M-H7.5, CN9 2X3F-H7.5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

Commit message: Fix Typo + Add Schematic as PDF
Schematic Typo Corrected.
Electrical Characteristic Updated.
Sunflower Shield PDF Schematic Added.
Parts:
- C31: value 2200pF -> 0.22uF
Other:
- note added: "250"
- note removed: "150"
Changed lines of the file:
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@@
 <setting verticaltext="up"/>
 </settings>
-<grid distance="0.1" unitdist="inch" unit="inch" style="lines" multiple="1" display="no" altdistance="0.01" altunitdist="inch" altunit="inch"/>
+<grid distance="0.1" unitdist="inch" unit="inch" style="lines" multiple="1" display="yes" altdistance="0.01" altunitdist="inch" altunit="inch"/>
 <layers>
 <layer number="1" name="Top" color="4" fill="1" visible="no" active="no"/>
@@
 <part name="R28" library="microbuilder" deviceset="RESISTOR" device="0805" value="2.37/1%"/>
 <part name="GND29" library="microbuilder" deviceset="GND" device=""/>
-<part name="C31" library="microbuilder" deviceset="CAP_CERAMIC" device="0603" value="2200pF"/>
+<part name="C31" library="microbuilder" deviceset="CAP_CERAMIC" device="0603" value="0.22uF"/>
 <part name="GND30" library="microbuilder" deviceset="GND" device=""/>
 <part name="H1" library="CowFish-Connectors" deviceset="MOUNTINGHOLE" device="3.2"/>
@@
 <text x="214.63" y="12.7" size="2.54" layer="94" align="bottom-center">mA</text>
 <text x="176.53" y="12.7" size="2.54" layer="94" align="bottom-center">-</text>
-<text x="189.23" y="12.7" size="2.54" layer="94" align="bottom-center">150</text>
+<text x="189.23" y="12.7" size="2.54" layer="94" align="bottom-center">250</text>
 <text x="201.93" y="12.7" size="2.54" layer="94" align="bottom-center">-</text>
 <text x="320.04" y="24.13" size="2.54" layer="94" font="vector">P. Bartek</text>
